Commit message: Refactor: Separate arm_driver from arm_sim and restructure packages

File: src/arm_description/urdf/robot.urdf (robot description, URDF)
Before this commit: robot my_robot, 12 links, 11 joints
Links:
- link base: geometry collision mesh filename=package://arm_description/meshes/base.stl scale=0.001 0.001 0.001; visual mesh filename=package://arm_description/meshes/base.stl scale=0.001 0.001 0.001
- link joint1: geometry collision mesh filename=package://arm_description/meshes/joint1.stl scale=0.001 0.001 0.001; visual mesh filename=package://arm_description/meshes/joint1.stl scale=0.001 0.001 0.001
- link joint2: geometry collision mesh filename=package://arm_description/meshes/joint2.stl scale=0.001 0.001 0.001; visual mesh filename=package://arm_description/meshes/joint2.stl scale=0.001 0.001 0.001
- link link1_1: geometry collision mesh filename=package://arm_description/meshes/link1_1.stl scale=0.001 0.001 0.001; visual mesh filename=package://arm_description/meshes/link1_1.stl scale=0.001 0.001 0.001
- link link1_2: geometry collision mesh filename=package://arm_description/meshes/link1_2.stl scale=0.001 0.001 0.001; visual mesh filename=package://arm_description/meshes/link1_2.stl scale=0.001 0.001 0.001
- link link1_3: geometry collision mesh filename=package://arm_description/meshes/link1_3.stl scale=0.001 0.001 0.001; visual mesh filename=package://arm_description/meshes/link1_3.stl scale=0.001 0.001 0.001
- link link2: geometry collision mesh filename=package://arm_description/meshes/link2.stl scale=0.001 0.001 0.001; visual mesh filename=package://arm_description/meshes/link2.stl scale=0.001 0.001 0.001
- link rs02_1: geometry collision mesh filename=package://arm_description/meshes/RS02(0.0.0).stl scale=0.001 0.001 0.001; visual mesh filename=package://arm_description/meshes/RS02(0.0.0).stl scale=0.001 0.001 0.001
- link rs02_2: geometry collision mesh filename=package://arm_description/meshes/RS02(0.0.0).stl scale=0.001 0.001 0.001; visual mesh filename=package://arm_description/meshes/RS02(0.0.0).stl scale=0.001 0.001 0.001
- link rs02_3: geometry collision mesh filename=package://arm_description/meshes/RS02(0.0.0).stl scale=0.001 0.001 0.001; visual mesh filename=package://arm_description/meshes/RS02(0.0.0).stl scale=0.001 0.001 0.001
- link rs03: geometry collision mesh filename=package://arm_description/meshes/RS03(0.0.0).stl scale=0.001 0.001 0.001; visual mesh filename=package://arm_description/meshes/RS03(0.0.0).stl scale=0.001 0.001 0.001
